Commit message: checkpoint: calibration depth pose improvements

File: urdf_rc5_right_hand/Robot_with_right_hand_cor.urdf (robot description, URDF)
Before this commit: robot rc5_aero_hand, 42 links, 41 joints
Joints:
- joint prehand_cam_to_d405_depth: origin xyz=0.009 0.0675 0.0912 rpy=0 -1.5707963267948966 -1.5707963267948966 -> xyz=0.009 0.0675 0.0912 rpy=0 1.5707963267948966 -1.5707963267948966

File: urdf_rc5_right_hand/urdf_with_simple_collisions.urdf (robot description, URDF)
Before this commit: robot rc5_aero_hand, 37 links, 36 joints
Joints:
- joint prehand_cam_to_d405_depth: origin xyz=0.009 0.0675 0.0912 rpy=0 -1.5707963267948966 -1.5707963267948966 -> xyz=0.009 0.0675 0.0912 rpy=0 1.5707963267948966 -1.5707963267948966
